File: hw/nucleo-lidar-breakout/nucleo-lidar-breakout.kicad_pcb (KiCad board)
At the start: 2 copper layers, 0 parts

Commit message: Released rplidar nucleo breakout v1.0 to oshpark
Parts:
- added C1: 0.1uF, Capacitor_SMD:C_0402_1005Metric, F.Cu at (76.8, 118.6)
- added C2: 10uF, Capacitor_SMD:C_0805_2012Metric, F.Cu at (106.5, 130.0)
- added C3: 100uF, Capacitor_SMD:C_1210_3225Metric, F.Cu at (106.0, 136.0)
- added C4: 0.1uF, Capacitor_SMD:C_0402_1005Metric, F.Cu at (76.8, 113.2)
- added J1: PJ-051AH, alvarop:PJ-051AH, F.Cu at (99.0, 99.0)
- added J2: ‎0532610471‎, alvarop:MOLEX_0532610471, F.Cu at (108.0, 139.0)
- added J3: ‎0532610371‎, alvarop:MOLEX_0532610371, F.Cu at (91.0, 139.0)
- added J4: 282834-3, TerminalBlock_TE-Connectivity:TerminalBlock_TE_282834-3_1x03_P2.54mm_Horizontal, F.Cu at (69.0, 112.5)
- added J5: Conn_01x03, Connector_PinHeader_2.54mm:PinHeader_1x03_P2.54mm_Vertical, F.Cu at (88.0, 105.5)
- added L1: 6.8uH, alvarop:BOURNS_SRN3015TA, F.Cu at (106.6, 127.0)
- added L2: 0.1uH, Inductor_SMD:L_0603_1608Metric, F.Cu at (107.4, 132.6)
- added Q1: Si7111EDN, Package_SO:Vishay_PowerPAK_1212-8_Single, F.Cu at (76.0, 107.0)
- added Q2: MMBT3904, Package_TO_SOT_SMD:SOT-23, F.Cu at (80.0, 110.0)
- added R1: 0.25, Resistor_SMD:R_0402_1005Metric, F.Cu at (106.2, 132.6)
- added R2: 100, Resistor_SMD:R_0402_1005Metric, F.Cu at (75.0, 115.0)
- added R3: 10k, Resistor_SMD:R_0402_1005Metric, F.Cu at (79.4, 113.2)
- added R4: 1k, Resistor_SMD:R_0402_1005Metric, F.Cu at (76.5, 110.0)
- added R5: 10k, Resistor_SMD:R_0402_1005Metric, F.Cu at (83.0, 111.0)
- added R6: 100, Resistor_SMD:R_0402_1005Metric, F.Cu at (109.0, 136.5)
- added R7: 100, Resistor_SMD:R_0402_1005Metric, F.Cu at (110.0, 136.5)
- added REF**: OSHW-Logo2_14.6x12mm_SilkScreen, Symbol:OSHW-Logo2_14.6x12mm_SilkScreen, F.Cu at (116.0, 102.0)
- added REF**: MountingHole_2.7mm_M2.5, MountingHole:MountingHole_2.7mm_M2.5, F.Cu at (120.0, 170.0)
- added REF**: MountingHole_2.7mm_M2.5, MountingHole:MountingHole_2.7mm_M2.5, F.Cu at (80.0, 170.0)
- added REF**: MountingHole_2.7mm_M2.5, MountingHole:MountingHole_2.7mm_M2.5, F.Cu at (72.0, 100.0)
- added REF**: MountingHole_2.7mm_M2.5, MountingHole:MountingHole_2.7mm_M2.5, F.Cu at (128.0, 100.0)
- added U1: TXS0101, alvarop:TI_SC70, F.Cu at (78.0, 116.0)
- added U2: NUCLEO_L476RG, alvarop:NUCLEO_L476RG, F.Cu at (100.0, 146.0)
Routing:
- net +5V: track 0.00 -> 95.4 mm
- net /LED_SIG: track 0.00 -> 67.1 mm, vias 0 -> 2
- net /LED_EN: track 0.00 -> 59.4 mm, vias 0 -> 2
- net Net-(R7-Pad1): track 0.00 -> 41.8 mm
- net /5V_USB: track 0.00 -> 41.2 mm
- net Net-(R6-Pad1): track 0.00 -> 35.3 mm
- net /LIDAR_EN: track 0.00 -> 34.2 mm
- net +3V3: track 0.00 -> 21.8 mm
- net GND: track 0.00 -> 17.3 mm, vias 0 -> 15
- net Net-(Q1-Pad4): track 0.00 -> 9.25 mm, vias 0 -> 2
- net /CLEAN_5V: track 0.00 -> 7.14 mm
- net /LED_SIG_OUT: track 0.00 -> 5.52 mm
- net Net-(C2-Pad1): track 0.00 -> 5.38 mm
- net Net-(R2-Pad1): track 0.00 -> 4.26 mm
- net /LIDAR_TX: track 0.00 -> 2.36 mm
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- added copper zone on F.Cu, net +5V
- added copper zone on F.Cu, net /5V_IN
- added copper zone on F.Cu, net /LED_5V_OUT
- added copper zone on B.Cu, net GND
Other:
- board outline added: 70 x 80 mm
- board text added: "5V SIG GND"
- board text added: "5V_IN"
- board text added: "5V_USB"
- board text added: "RPLidar Nucleo Breakout"
- board text added: "by @alvaroprieto"
- board text added: "v1.0"
