File: hw/nucleo-lidar-breakout/nucleo-lidar-breakout.sch (KiCad schematic (older format))
At the start: 22 parts, among them J1 PJ-051AH, J2 ‎0532610471‎, J3 ‎0532610371‎, J4 282834-3, J5 Conn_01x03, Q1 Si7111EDN, Q2 MMBT3904, U1 TXS0101, U2 NUCLEO_L476RG

Commit message: Add part numbers to schematic
Parts:
- C1, C4: DKPN (none) -> 490-1318-1-ND; MPN (none) -> GRM155R61A104KA01D
- C2: DKPN (none) -> 490-6473-1-ND‎; MPN (none) -> ‎GRM21BR61C106KE15K‎
- C3: DKPN (none) -> 1276-3364-1-ND‎; MPN (none) -> ‎CL32A107MPVNNNE‎
- J1: DKPN (none) -> CP-051AH-ND‎; MPN (none) -> ‎PJ-051AH‎
- J2: DKPN (none) -> WM7622CT-ND‎; MPN (none) -> ‎0532610471‎
- J3: DKPN (none) -> WM7621CT-ND‎; MPN (none) -> ‎0532610371‎
- L1: DKPN (none) -> SRN3015TA-6R8MCT-ND‎; MPN (none) -> ‎SRN3015TA-6R8M‎
- L2: DKPN (none) -> ‎445-6386-1-ND‎; MPN (none) -> ‎MLZ1608DR10DT000‎
- Q1: DKPN (none) -> SI7111EDN-T1-GE3CT-ND‎; MPN (none) -> ‎SI7111EDN-T1-GE3‎
- Q2: DKPN (none) -> MMBT3904LT3GOSCT-ND‎; MPN (none) -> ‎MMBT3904LT3G‎
- R1: DKPN (none) -> CSR0402FKR250CT-ND‎; MPN (none) -> ‎CSR0402FKR250‎
- R2, R6, R7: DKPN (none) -> 311-100LRCT-ND; MPN (none) -> RC0402FR-07100RL
- R3, R5: DKPN (none) -> 311-10KJRCT-ND; MPN (none) -> RC0402JR-0710KL
- R4: DKPN (none) -> A106129TR-ND; MPN (none) -> CRG0402J1K0
- U1: DKPN (none) -> 296-22864-1-ND‎; MPN (none) -> ‎TXS0101DCKR‎
Changed lines of the file:
@@
 F 2 "alvarop:MOLEX_0532610371" H 10500 2000 50  0001 C CNN
 F 3 "~" H 10500 2000 50  0001 C CNN
+F 4 "WM7621CT-ND‎" H 10500 2000 50  0001 C CNN "DKPN"
+F 5 "‎0532610371‎" H 10500 2000 50  0001 C CNN "MPN"
 	1    10500 2000
 	1    0    0    -1
@@
 F 2 "alvarop:MOLEX_0532610471" H 10500 1200 50  0001 C CNN
 F 3 "~" H 10500 1200 50  0001 C CNN
+F 4 "WM7622CT-ND‎" H 10500 1200 50  0001 C CNN "DKPN"
+F 5 "‎0532610471‎" H 10500 1200 50  0001 C CNN "MPN"
 	1    10500 1200
 	1    0    0    1
@@
 F 2 "alvarop:TI_SC70" H 5300 1400 50  0001 C CNN
 F 3 "" H 5300 1400 50  0001 C CNN
+F 4 "296-22864-1-ND‎" H 5300 1400 50  0001 C CNN "DKPN"
+F 5 "‎TXS0101DCKR‎" H 5300 1400 50  0001 C CNN "MPN"
 	1    5300 1400
 	1    0    0    -1
@@
 F 2 "Resistor_SMD:R_0402_1005Metric" H 6100 1700 50  0001 C CNN
 F 3 "~" H 6100 1700 50  0001 C CNN
+F 4 "311-10KJRCT-ND" H 6100 1700 50  0001 C CNN "DKPN"
+F 5 "RC0402JR-0710KL" H 6100 1700 50  0001 C CNN "MPN"
 	1    6100 1700
 	1    0    0    -1
@@
 F 2 "Resistor_SMD:R_0402_1005Metric" H 5800 1700 50  0001 C CNN
 F 3 "~" H 5800 1700 50  0001 C CNN
+F 4 "311-100LRCT-ND" H 5800 1700 50  0001 C CNN "DKPN"
+F 5 "RC0402FR-07100RL" H 5800 1700 50  0001 C CNN "MPN"
 	1    5800 1700
 	1    0    0    -1
@@
 F 2 "Capacitor_SMD:C_0402_1005Metric" H 6600 1600 50  0001 C CNN
 F 3 "~" H 6600 1600 50  0001 C CNN
+F 4 "490-1318-1-ND" H 6600 1600 50  0001 C CNN "DKPN"
+F 5 "GRM155R61A104KA01D" H 6600 1600 50  0001 C CNN "MPN"
 	1    6600 1600
 	1    0    0    -1
@@
 F 2 "Capacitor_SMD:C_0402_1005Metric" H 4100 1500 50  0001 C CNN
 F 3 "~" H 4100 1500 50  0001 C CNN
+F 4 "490-1318-1-ND" H 4100 1500 50  0001 C CNN "DKPN"
+F 5 "GRM155R61A104KA01D" H 4100 1500 50  0001 C CNN "MPN"
 	1    4100 1500
 	1    0    0    -1
@@
 F 2 "Package_TO_SOT_SMD:SOT-23" H 9600 3925 50  0001 L CIN
 F 3 "https://www.fairchildsemi.com/datasheets/2N/2N3904.pdf" H 9400 4000 50  0001 L CNN
+F 4 "MMBT3904LT3GOSCT-ND‎" H 9400 4000 50  0001 C CNN "DKPN"
+F 5 "‎MMBT3904LT3G‎" H 9400 4000 50  0001 C CNN "MPN"
 	1    9400 4000
 	1    0    0    -1
@@
 F 2 "Package_SO:Vishay_PowerPAK_1212-8_Single" H 10100 3525 50  0001 L CIN
 F 3 "http://www.vishay.com/docs/67807/si7111edn.pdf" V 9900 3600 50  0001 L CNN
+F 4 "SI7111EDN-T1-GE3CT-ND‎" H 9900 3600 50  0001 C CNN "DKPN"
+F 5 "‎SI7111EDN-T1-GE3‎" H 9900 3600 50  0001 C CNN "MPN"
 	1    9900 3600
 	1    0    0    -1
@@
 F 2 "Resistor_SMD:R_0402_1005Metric" H 9000 4000 50  0001 C CNN
 F 3 "~" H 9000 4000 50  0001 C CNN
+F 4 "311-10KJRCT-ND" H 9000 4000 50  0001 C CNN "DKPN"
+F 5 "RC0402JR-0710KL" H 9000 4000 50  0001 C CNN "MPN"
 	1    9000 4000
 	0    1    1    0
@@
 F 2 "Resistor_SMD:R_0402_1005Metric" H 9700 3200 50  0001 C CNN
 F 3 "~" H 9700 3200 50  0001 C CNN
+F 4 "A106129TR-ND" H 9700 3200 50  0001 C CNN "DKPN"
+F 5 "CRG0402J1K0" H 9700 3200 50  0001 C CNN "MPN"
 	1    9700 3200
 	0    1    1    0
@@
 F 2 "Resistor_SMD:R_0402_1005Metric" H 5600 4600 50  0001 C CNN
 F 3 "~" H 5600 4600 50  0001 C CNN
+F 4 "311-100LRCT-ND" H 5600 4600 50  0001 C CNN "DKPN"
+F 5 "RC0402FR-07100RL" H 5600 4600 50  0001 C CNN "MPN"
 	1    5600 4600
 	0    1    1    0
@@
 F 2 "Resistor_SMD:R_0402_1005Metric" H 5600 5200 50  0001 C CNN
 F 3 "~" H 5600 5200 50  0001 C CNN
+F 4 "311-100LRCT-ND" H 5600 5200 50  0001 C CNN "DKPN"
+F 5 "RC0402FR-07100RL" H 5600 5200 50  0001 C CNN "MPN"
 	1    5600 5200
 	0    1    1    0
@@
 F 2 "alvarop:PJ-051AH" H 1450 1160 50  0001 C CNN
 F 3 "~" H 1450 1160 50  0001 C CNN
+F 4 "CP-051AH-ND‎" H 1400 1200 50  0001 C CNN "DKPN"
+F 5 "‎PJ-051AH‎" H 1400 1200 50  0001 C CNN "MPN"
 	1    1400 1200
 	1    0    0    -1
@@
 F 2 "Capacitor_SMD:C_0805_2012Metric" H 8900 1500 50  0001 C CNN
 F 3 "~" H 8900 1500 50  0001 C CNN
+F 4 "490-6473-1-ND‎" H 8900 1500 50  0001 C CNN "DKPN"
+F 5 "‎GRM21BR61C106KE15K‎" H 8900 1500 50  0001 C CNN "MPN"
 	1    8900 1500
 	1    0    0    -1
@@
 F 2 "Capacitor_SMD:C_1210_3225Metric" H 9500 1500 50  0001 C CNN
 F 3 "~" H 9500 1500 50  0001 C CNN
+F 4 "1276-3364-1-ND‎" H 9500 1500 50  0001 C CNN "DKPN"
+F 5 "‎CL32A107MPVNNNE‎" H 9500 1500 50  0001 C CNN "MPN"
 	1    9500 1500
 	1    0    0    -1
@@
 F 2 "alvarop:BOURNS_SRN3015TA" H 8600 1200 50  0001 C CNN
 F 3 "~" H 8600 1200 50  0001 C CNN
+F 4 "SRN3015TA-6R8MCT-ND‎" H 8600 1200 50  0001 C CNN "DKPN"
+F 5 "‎SRN3015TA-6R8M‎" H 8600 1200 50  0001 C CNN "MPN"
 	1    8600 1200
 	0    -1   -1   0
@@
 F 2 "Inductor_SMD:L_0603_1608Metric" H 9200 1200 50  0001 C CNN
 F 3 "~" H 9200 1200 50  0001 C CNN
+F 4 "‎445-6386-1-ND‎" H 9200 1200 50  0001 C CNN "DKPN"
+F 5 "‎MLZ1608DR10DT000‎" H 9200 1200 50  0001 C CNN "MPN"
 	1    9200 1200
 	0    -1   -1   0
@@
 F 2 "Resistor_SMD:R_0402_1005Metric" H 9200 900 50  0001 C CNN
 F 3 "~" H 9200 900 50  0001 C CNN
+F 4 "CSR0402FKR250CT-ND‎" H 9200 900 50  0001 C CNN "DKPN"
+F 5 "‎CSR0402FKR250‎" H 9200 900 50  0001 C CNN "MPN"
 	1    9200 900
 	0    1    1    0
